File: pcb/micro discord board.kicad_sch (KiCad schematic)
At the start: 9 parts, among them SW1 SW_Push, SW2 SW_Push, SW3 SW_Push, SW4 SW_Push, SW5 RotaryEncoder, U1 XIAO-RP2040-DIP

Commit message: Add files via upload
Parts:
- removed DS1: OLED-128O064D, Display:OLED-128O064D, symbol Seeed_Studio_XIAO_Series:OLED-128O064D
- removed U1: XIAO-RP2040-DIP, Package_DIP:DIP-14_W7.62mm, symbol Seeed_Studio_XIAO_Series:XIAO-RP2040-DIP
- added U1: XIAO-RP2040-SMD, Hackclub Footprints:XIAO-RP2040-DIP, symbol Seeed_Studio_XIAO_Series:XIAO-RP2040-SMD
- added U2: OLED_0.91_128x32, Hackclub Footprints:OLED_0.91_128x32, symbol Hackclub Symbols:OLED_0.91_128x32
Connections:
- net +5V: now also U1.14 (5V), U2.2 (VCC)
- net GND: now also U1.13 (GND), U2.1 (GND)
- net at SW4.2: now also U1.4 (GPIO29_A3_D3)
- net at SW3.2: now also U1.3 (GPIO28_A2_D2)
- net at SW2.2: now also U1.2 (GPIO27_A1_D1)
- net at SW1.2: now also U1.1 (GPIO26_A0_D0)
- net at D1.3 (DIN): now also U1.8 (GPIO1_D7_CSn_RX)
- net at SW5.B: now also U1.6 (GPIO7_D5_SCL)
- net at SW5.A: now also U1.5 (GPIO6_D4_SDA)
- new net: U1.10 (GPIO4_D9_MISO), U2.4 (SDA)
- new net: U1.11 (GPIO3_D10_MOSI), U2.3 (SCL)
